Commit message: Update centauro_tray

File: robolearn_envs/pybullet/common/surfaces/models/plane/plane_checker_blue.urdf (robot description, URDF)
Before this commit: robot plane, 1 links, 0 joints
Links:
- link planeLink: geometry collision box size=100 100 10; visual mesh filename=plane_checker_blue.obj scale=1 1 1

File: robolearn_envs/robot_models/hyq/hyq_lf_lh_rf_rh.urdf (robot description, URDF)
Before this commit: robot hyq, 13 links, 12 joints
Links:
- link trunk: mass 58.96 -> 10.00
